File: Duophonic/pitchdac.brd (EAGLE design)
At the start: 55.8 x 29.7 mm, 30 parts, among them IC1 AD5781ARUZ, U1 opa2186, U2 opa2186

Commit message: correct stupid error
Parts:
- removed C1: 1nf, rcl:C0805K
- removed C2: 1nF, rcl:C0805K
- added C101, C201: 22pF, rcl:C0805K
- added R6: 220R, rcl:R0805W
- added R7: 10k, rcl:R0805W
- R1, R2: value 220R -> 10k 0.02% 5ppm
- R3: value 4k7 -> 220R
- R4: value 4k7 -> 10k 0.02% 5ppm
- R5: value 10k -> 10k 0.02% 5ppm
- moved R5 39.6 mm to (50.8, 7.62), turned to 0 degrees
- moved R2 14.9 mm to (52.1, 24.1)
- moved R3 14.9 mm to (52.1, 21.6)
- moved R4 14.0 mm to (39.6, 13.1)
- moved R1 10.5 mm to (39.6, 15.6)
- moved C12 5.86 mm to (41.0, 20.1), turned to 270 degrees
- moved C13 3.81 mm to (52.1, 16.5)
- moved C7 3.81 mm to (49.5, 15.2)
- moved PITCH 3.81 mm to (61.0, 14.0)
- moved U2 3.05 mm to (45.0, 15.2)
- moved C6 0.28 mm to (38.2, 20.1)
Connections:
- new net N$2: R1.2, U2.3
- new net N$3: R4.2, U2.5
- net 3V3: now also R7.2; no longer R5.2
- net N$1: now also C201.2, R5.1; no longer C1.2, R3.1
- net N$15: now also C201.1, R6.1; no longer C1.1, R2.1
- net N$16: now also C101.1, R3.1; no longer C2.1, R1.1
- net N$5: now also C101.2, R2.1; no longer C2.2, R4.1
- net PITCH1: now also R2.2, R3.2; no longer R1.2, R4.2
- net PITCH2: now also R5.2, R6.2; no longer R2.2, R3.2
- net SYNC: now also R7.1; no longer R5.1
- net UNBUF: now also R1.1, R4.1; no longer U2.3, U2.5
Routing:
- net N$2: track 0.00 -> 5.82 mm
- net UNBUF: track 28.7 -> 23.8 mm
- net +9V5: track 120.3 -> 124.9 mm
- net N$3: track 0.00 -> 2.56 mm
- net -9V5: track 67.5 -> 69.4 mm
- net AGND: track 57.4 -> 58.9 mm
- net N$1: track 9.61 -> 10.2 mm
Other:
- board size 55.8 x 29.7 mm -> 60.9 x 29.7 mm

Commit message: idiot!!!
Parts:
- removed R1, R4: 10k 0.02% 5ppm, rcl:R0805W
- C101, C201: value 22pF -> 100pF
- R2, R5: value 10k 0.02% 5ppm -> 4k7
Connections:
- removed net N$2: R1.2, U2.3
- removed net N$3: R4.2, U2.5
- net UNBUF: now also U2.3, U2.5; no longer R1.1, R4.1
Routing:
- net UNBUF: track 23.8 -> 31.8 mm
- net N$2: track 5.82 -> 0.00 mm
- net N$3: track 2.56 -> 0.00 mm
Other:
- board size 60.9 x 29.7 mm -> 59.9 x 29.7 mm
