File: Duophonic/KiCad/PerfDac_v02_extbuf/PerfDac_v02_extbuf.kicad_sch (KiCad schematic)
At the start: 12 parts, among them IC1 SN74AHCT125QDRQ1, IC2 DAC8168ICPW, J1 Conn_01x06_Socket, J2 Conn_01x06_Socket

Commit message: finish PerfDAC v0.2 board
Parts:
- removed J1: Conn_01x06_Socket, symbol Connector:Conn_01x06_Socket
- removed PWR1: Conn_01x04_Pin, Connector_PinHeader_2.54mm:PinHeader_1x04_P2.54mm_Vertical, symbol Connector:Conn_01x04_Pin
- added J2: Conn_01x06_Socket, Connector_PinSocket_2.54mm:PinSocket_1x06_P2.54mm_Vertical, symbol Connector:Conn_01x06_Socket
- J1: renamed from J2; footprint (none) -> Connector_PinSocket_2.54mm:PinSocket_1x06_P2.54mm_Vertical
Connections:
- net +5V: now also J1.3 (Pin_3), J2.3 (Pin_3)
- net GND: now also J1.6 (Pin_6), J2.6 (Pin_6)
- net VOUT_A: now also J1.5 (Pin_5)
- net VOUT_B: now also J2.5 (Pin_5)
- net VOUT_C: now also J1.4 (Pin_4)
- net VOUT_D: now also J2.4 (Pin_4)
- net VOUT_E: now also J1.2 (Pin_2)
- net VOUT_F: now also J2.2 (Pin_2)
- net VOUT_G: now also J1.1 (Pin_1)
- net VOUT_H: now also J2.1 (Pin_1)
Other:
- moved on the sheet: C1, C2, C3, C4, IC1, IC2, J1, R1, R2, SPI1
